Commit message: Add files via upload

File: urdf/p60_v2.urdf (robot description, URDF)
Before this commit: robot robot_P60_v2, 7 links, 6 joints
Links:
- link back_wheel: geometry collision cylinder length=0.1 radius=0.2; visual cylinder length=0.1 radius=0.2
- link base_link: geometry collision box size=0.5 0.5 0.25; visual box size=0.5 0.5 0.25
- link front_wheel: geometry collision cylinder length=0.1 radius=0.2; visual cylinder length=0.1 radius=0.2
- link left_wheel: geometry collision cylinder length=0.1 radius=0.2; visual cylinder length=0.1 radius=0.2
- link right_wheel: geometry collision cylinder length=0.1 radius=0.2; visual cylinder length=0.1 radius=0.2
Joints:
- joint joint_back_wheel: parent base_wheel_steer -> back_wheel_steer
- joint joint_back_wheel_steer: limit (none) -> lower=-1.0 upper=1.0 effort=1000.0 velocity=0.5
- joint joint_front_wheel_steer: limit (none) -> lower=-1.0 upper=1.0 effort=1000.0 velocity=0.5
